File: MINI VESC.sch (KiCad schematic (older format))
At the start: 151 parts, among them P1 CONN_1, P10 CONN_01X06, P11 CONN_01X06, P2 CONN_1, P3 CONN_1, P4 CONN_1, P5 CONN_1, P6 CONN_1, P9 CONN_01X06, Q1 NTMFS5C604NLT1G, Q2 NTMFS5C604NLT1G, Q3 NTMFS5C604NLT1G, Q4 NTMFS5C604NLT1G, Q5 NTMFS5C604NLT1G, Q6 NTMFS5C604NLT1G, U1 LM5113SDE, U10 MCP1700, U2 LM5113SDE, U3 LM5113SDE, U4 AD8417, U5 AD8417, U6 AD8417, U7 STM32F405RGT6, U8 LMR16006YDDCT, U9 MCP1700, X1 ABM3B-8.000MHZ

Commit message: cap
Parts:
- C80: value 2u2 100V 56x -> 10u
Other:
- note added: "56x 2u2 100V"
Changed lines of the file:
@@
 LIBS:contrib
 LIBS:valves
-LIBS:mojaKniznica
-LIBS:kniznica-kicad
-LIBS:BLDC_4-cache
-LIBS:open-project
 LIBS:MINI VESC-cache
 EELAYER 25 0
@@
 P 5000 5800
 F 0 "C80" H 5000 5700 50  0000 L CNN
-F 1 "2u2 100V 56x" H 5100 6000 50  0000 L CNN
+F 1 "10u" H 5100 6000 50  0001 L CNN
 F 2 "Resistors_SMD:R_1206" H 5038 5650 50  0001 C CNN
 F 3 "" H 5000 5800 50  0000 C CNN
@@
 Wire Wire Line
 	2200 4550 2250 4550
+Text Notes 5150 5600 0    60   ~ 0
+56x 2u2 100V
 $EndSCHEMATC

Commit message: new kicad port
3d models change
Parts:
- C1, C10, C11, C12, C13, C14, C15, C16, C17, C18, C19, C2, C20, C21, C22, C23, C24, C25, C26, C27, C28, C29, C3, C30, C31, C32, C33, C34, C35, C36, C37, C38, C39, C4, C40, C41, C42, C43, C44, C45, C46, C47, C48, C49, C5, C50, C51, C52, C53, C54, C55, C56, C57, C58, C59, C6, C60, C61, C62, C63, C64, C65, C66, C67, C68, C69, C7, C70, C71, C72, C73, C74, C75, C76, C77, C78, C79, C8, C80, C81, C82, C83, C84, C85, C86, C87, C88, C89, C9, C90: symbol C -> device:C
- D1: symbol D_Schottky -> device:D_Schottky
- D3, D4: symbol LED -> device:LED
- L1: symbol INDUCTOR -> MINI~VESC-rescue:INDUCTOR-RESCUE-MINI_VESC
- P1, P2, P3, P4, P5, P6: symbol CONN_1 -> MINI~VESC-rescue:CONN_1-RESCUE-MINI_VESC
- P10, P11, P9: symbol CONN_01X06 -> conn:CONN_01X06
- Q1, Q2, Q3, Q4, Q5, Q6: symbol Q_NMOS_GSD -> device:Q_NMOS_GSD
- R1, R2, R3: symbol RSENS -> MINI~VESC-rescue:RSENS-RESCUE-MINI_VESC
- R10, R11, R12, R13, R14, R15, R16, R17, R18, R19, R20, R21, R22, R25, R27, R28, R29, R30, R31, R32, R33, R34, R4, R5, R6, R7, R8, R9: symbol R -> device:R
- U1, U2, U3: symbol LM5001 -> MINI~VESC-rescue:LM5001-RESCUE-MINI_VESC
- U10, U9: symbol MCP1700 -> MINI~VESC-rescue:MCP1700-RESCUE-MINI_VESC
- U4, U5, U6: symbol AD8418 -> MINI~VESC-rescue:AD8418-RESCUE-MINI_VESC
- U7: symbol STM32F40X_LQFP64 -> MINI~VESC-rescue:STM32F40X_LQFP64-RESCUE-MINI_VESC
- U8: symbol BD9G101G -> MINI~VESC-rescue:BD9G101G-RESCUE-MINI_VESC
- X1: symbol CRYSTAL_SMD -> MINI~VESC-rescue:CRYSTAL_SMD-RESCUE-MINI_VESC

Commit message: update lib/sch to use kicad5 default library names/parts
Parts:
- C1, C10, C11, C12, C13, C14, C15, C16, C17, C18, C19, C2, C20, C21, C22, C23, C24, C25, C26, C27, C28, C29, C3, C30, C31, C32, C33, C34, C35, C36, C37, C38, C39, C4, C40, C41, C42, C43, C44, C45, C46, C47, C48, C49, C5, C50, C51, C52, C53, C54, C55, C56, C57, C58, C59, C6, C60, C61, C62, C63, C64, C65, C66, C67, C68, C69, C7, C70, C71, C72, C73, C74, C75, C76, C77, C78, C79, C8, C80, C81, C82, C83, C84, C85, C86, C87, C88, C89, C9, C90: symbol device:C -> Device:C
- D1: symbol device:D_Schottky -> Device:D_Schottky
- D3, D4: symbol device:LED -> Device:LED
- P10, P11, P9: value CONN_01X06 -> Conn_01x06; symbol conn:CONN_01X06 -> Connector_Generic:Conn_01x06
- Q1, Q2, Q3, Q4, Q5, Q6: symbol device:Q_NMOS_GSD -> Device:Q_NMOS_GSD
- R10, R11, R12, R13, R14, R15, R16, R17, R18, R19, R20, R21, R22, R25, R27, R28, R29, R30, R31, R32, R33, R34, R4, R5, R6, R7, R8, R9: symbol device:R -> Device:R
Connections:
- wire segments 497 -> 574
